File: DifferentialProbe.sch (KiCad schematic (older format))
At the start: 56 parts, among them J10 Conn_01x01, J11 Conn_01x01, J12 Conn_01x01, J13 Conn_01x01, J16 Conn_01x01, J17 Conn_01x01, J18 Conn_Coaxial, J6 Conn_01x01, J7 Conn_01x01, Q10 2SC3356, Q11 2SC3356, Q12 2SC3356, Q13 2SC3356, Q14 2SC3356, Q15 2SC3356, Q9 2SC3356

Commit message: JLCPCB order 2020-05-20
Parts:
- R43, R44, R62: value 220R -> 22R; LCSC C17557 -> C17561
Changed lines of the file:
@@
 $EndComp
 $Comp
-L GND #PWR48
+L GND #PWR044
 U 1 1 5EB7DC05
 P 2200 4650
-F 0 "#PWR48" H 2200 4400 50  0001 C CNN
+F 0 "#PWR044" H 2200 4400 50  0001 C CNN
 F 1 "GND" H 2200 4500 50  0000 C CNN
 F 2 "" H 2200 4650 50  0001 C CNN
@@
 $EndComp
 $Comp
-L GND #PWR55
+L GND #PWR045
 U 1 1 5EB7DC0C
 P 3100 2550
-F 0 "#PWR55" H 3100 2300 50  0001 C CNN
+F 0 "#PWR045" H 3100 2300 50  0001 C CNN
 F 1 "GND" H 3100 2400 50  0000 C CNN
 F 2 "" H 3100 2550 50  0001 C CNN
@@
 $EndComp
 $Comp
-L GND #PWR44
+L GND #PWR046
 U 1 1 5EB7DC0E
 P 1350 3600
-F 0 "#PWR44" H 1350 3350 50  0001 C CNN
+F 0 "#PWR046" H 1350 3350 50  0001 C CNN
 F 1 "GND" H 1350 3450 50  0000 C CNN
 F 2 "" H 1350 3600 50  0001 C CNN
@@
 $EndComp
 $Comp
-L GND #PWR46
+L GND #PWR047
 U 1 1 5EB7DC14
 P 2200 2500
-F 0 "#PWR46" H 2200 2250 50  0001 C CNN
+F 0 "#PWR047" H 2200 2250 50  0001 C CNN
 F 1 "GND" H 2200 2350 50  0000 C CNN
 F 2 "" H 2200 2500 50  0001 C CNN
@@
 $EndComp
 $Comp
-L GND #PWR51
+L GND #PWR048
 U 1 1 5EB7DC1C
 P 2550 3600
-F 0 "#PWR51" H 2550 3350 50  0001 C CNN
+F 0 "#PWR048" H 2550 3350 50  0001 C CNN
 F 1 "GND" H 2550 3450 50  0000 C CNN
 F 2 "" H 2550 3600 50  0001 C CNN
@@
 $EndComp
 $Comp
-L GND #PWR65
+L GND #PWR049
 U 1 1 5EB7DC1D
 P 5700 5200
-F 0 "#PWR65" H 5700 4950 50  0001 C CNN
+F 0 "#PWR049" H 5700 4950 50  0001 C CNN
 F 1 "GND" H 5700 5050 50  0000 C CNN
 F 2 "" H 5700 5200 50  0001 C CNN
@@
 $EndComp
 $Comp
-L GND #PWR69
+L GND #PWR050
 U 1 1 5EB7DC20
 P 7200 5150
-F 0 "#PWR69" H 7200 4900 50  0001 C CNN
+F 0 "#PWR050" H 7200 4900 50  0001 C CNN
 F 1 "GND" H 7200 5000 50  0000 C CNN
 F 2 "" H 7200 5150 50  0001 C CNN
@@
 $EndComp
 $Comp
-L GND #PWR59
+L GND #PWR051
 U 1 1 5EB7DC21
 P 3500 1900
-F 0 "#PWR59" H 3500 1650 50  0001 C CNN
+F 0 "#PWR051" H 3500 1650 50  0001 C CNN
 F 1 "GND" H 3500 1750 50  0000 C CNN
 F 2 "" H 3500 1900 50  0001 C CNN
@@
 $EndComp
 $Comp
-L GND #PWR50
+L GND #PWR052
 U 1 1 5EB7DC27
 P 2200 6550
-F 0 "#PWR50" H 2200 6300 50  0001 C CNN
+F 0 "#PWR052" H 2200 6300 50  0001 C CNN
 F 1 "GND" H 2200 6400 50  0000 C CNN
 F 2 "" H 2200 6550 50  0001 C CNN
@@
 $EndComp
 $Comp
-L GND #PWR45
+L GND #PWR053
 U 1 1 5EB7DC2C
 P 1350 5500
-F 0 "#PWR45" H 1350 5250 50  0001 C CNN
+F 0 "#PWR053" H 1350 5250 50  0001 C CNN
 F 1 "GND" H 1350 5350 50  0000 C CNN
 F 2 "" H 1350 5500 50  0001 C CNN
@@
 $EndComp
 $Comp
-L GND #PWR52
+L GND #PWR054
 U 1 1 5EB7DC2F
 P 2550 5500
-F 0 "#PWR52" H 2550 5250 50  0001 C CNN
+F 0 "#PWR054" H 2550 5250 50  0001 C CNN
 F 1 "GND" H 2550 5350 50  0000 C CNN
 F 2 "" H 2550 5500 50  0001 C CNN
@@
 	3550 5600 3550 5400
 $Comp
-L GND #PWR57
+L GND #PWR055
 U 1 1 5EB7DC31
 P 3250 5850
-F 0 "#PWR57" H 3250 5600 50  0001 C CNN
+F 0 "#PWR055" H 3250 5600 50  0001 C CNN
 F 1 "GND" H 3250 5700 50  0000 C CNN
 F 2 "" H 3250 5850 50  0001 C CNN
@@
 	3650 5600 3550 5600
 $Comp
-L GND #PWR61
+L GND #PWR056
 U 1 1 5EB7DC32
 P 3950 5850
-F 0 "#PWR61" H 3950 5600 50  0001 C CNN
+F 0 "#PWR056" H 3950 5600 50  0001 C CNN
 F 1 "GND" H 3950 5700 50  0000 C CNN
 F 2 "" H 3950 5850 50  0001 C CNN
@@
 	6050 3850 6050 3750
 $Comp
-L GND #PWR66
+L GND #PWR057
 U 1 1 5EB7DC3C
 P 6050 3850
-F 0 "#PWR66" H 6050 3600 50  0001 C CNN
+F 0 "#PWR057" H 6050 3600 50  0001 C CNN
 F 1 "GND" H 6050 3700 50  0000 C CNN
 F 2 "" H 6050 3850 50  0001 C CNN
@@
 	2900 5200 2900 5100
 $Comp
-L GND #PWR53
+L GND #PWR058
 U 1 1 5EB7DC3E
 P 2900 5200
-F 0 "#PWR53" H 2900 4950 50  0001 C CNN
+F 0 "#PWR058" H 2900 4950 50  0001 C CNN
 F 1 "GND" H 2900 5050 50  0000 C CNN
 F 2 "" H 2900 5200 50  0001 C CNN
@@
 Connection ~ 4650 3650
 $Comp
-L GND #PWR63
+L GND #PWR059
 U 1 1 5EB7DC46
 P 5000 3700
-F 0 "#PWR63" H 5000 3450 50  0001 C CNN
+F 0 "#PWR059" H 5000 3450 50  0001 C CNN
 F 1 "GND" H 5000 3550 50  0000 C CNN
 F 2 "" H 5000 3700 50  0001 C CNN
@@
 Connection ~ 3350 3650
 $Comp
-L GND #PWR60
+L GND #PWR060
 U 1 1 5EB7DC4A
 P 3700 3700
-F 0 "#PWR60" H 3700 3450 50  0001 C CNN
+F 0 "#PWR060" H 3700 3450 50  0001 C CNN
 F 1 "GND" H 3700 3550 50  0000 C CNN
 F 2 "" H 3700 3700 50  0001 C CNN
@@
 $EndComp
 $Comp
-L GND #PWR67
+L GND #PWR061
 U 1 1 5EB7DC53
 P 6350 5200
-F 0 "#PWR67" H 6350 4950 50  0001 C CNN
+F 0 "#PWR061" H 6350 4950 50  0001 C CNN
 F 1 "GND" H 6350 5050 50  0000 C CNN
 F 2 "" H 6350 5200 50  0001 C CNN
@@
 $EndComp
 $Comp
-L GND #PWR68
+L GND #PWR062
 U 1 1 5EB7DC55
 P 6800 5200
-F 0 "#PWR68" H 6800 4950 50  0001 C CNN
+F 0 "#PWR062" H 6800 4950 50  0001 C CNN
 F 1 "GND" H 6800 5050 50  0000 C CNN
 F 2 "" H 6800 5200 50  0001 C CNN
@@
 P 1550 3950
 F 0 "R43" V 1650 3950 50  0000 C CNN
-F 1 "220R" V 1550 3950 50  0000 C CNN
+F 1 "22R" V 1550 3950 50  0000 C CNN
 F 2 "Resistors_SMD:R_0805_HandSoldering" V 1480 3950 50  0001 C CNN
 F 3 "" H 1550 3950 50  0001 C CNN
-F 4 "C17557" V 1550 3950 60  0001 C CNN "LCSC"
+F 4 "C17561" V 1550 3950 60  0001 C CNN "LCSC"
 	1    1550 3950
 	0    1    1    0
@@
 P 1550 5850
 F 0 "R44" V 1650 5850 50  0000 C CNN
-F 1 "220R" V 1550 5850 50  0000 C CNN
+F 1 "22R" V 1550 5850 50  0000 C CNN
 F 2 "Resistors_SMD:R_0805_HandSoldering" V 1480 5850 50  0001 C CNN
 F 3 "" H 1550 5850 50  0001 C CNN
-F 4 "C17557" V 1550 5850 60  0001 C CNN "LCSC"
+F 4 "C17561" V 1550 5850 60  0001 C CNN "LCSC"
 	1    1550 5850
 	0    1    1    0
@@
 P 5200 4250
 F 0 "R62" V 5280 4250 50  0000 C CNN
-F 1 "220R" V 5200 4250 50  0000 C CNN
+F 1 "22R" V 5200 4250 50  0000 C CNN
 F 2 "Resistors_SMD:R_0805_HandSoldering" V 5130 4250 50  0001 C CNN
 F 3 "" H 5200 4250 50  0001 C CNN
-F 4 "C17557" V 5200 4250 60  0001 C CNN "LCSC"
+F 4 "C17561" V 5200 4250 60  0001 C CNN "LCSC"
 	1    5200 4250
 	0    1    1    0
@@
 	5050 4250 5000 4250
 $Comp
-L +BATT #PWR54
+L +BATT #PWR063
 U 1 1 5EB77B79
 P 3100 1500
-F 0 "#PWR54" H 3100 1350 50  0001 C CNN
+F 0 "#PWR063" H 3100 1350 50  0001 C CNN
 F 1 "+BATT" H 3100 1640 50  0000 C CNN
 F 2 "" H 3100 1500 50  0001 C CNN
@@
 $EndComp
 $Comp
-L +BATT #PWR47
+L +BATT #PWR064
 U 1 1 5EB77C65
 P 2200 3050
-F 0 "#PWR47" H 2200 2900 50  0001 C CNN
+F 0 "#PWR064" H 2200 2900 50  0001 C CNN
 F 1 "+BATT" H 2200 3190 50  0000 C CNN
 F 2 "" H 2200 3050 50  0001 C CNN
@@
 	2200 3050 2200 3100
 $Comp
-L +BATT #PWR58
+L +BATT #PWR065
 U 1 1 5EB77FC8
 P 3350 3300
-F 0 "#PWR58" H 3350 3150 50  0001 C CNN
+F 0 "#PWR065" H 3350 3150 50  0001 C CNN
 F 1 "+BATT" H 3350 3440 50  0000 C CNN
 F 2 "" H 3350 3300 50  0001 C CNN
@@
 $EndComp
 $Comp
-L +BATT #PWR62
+L +BATT #PWR066
 U 1 1 5EB78125
 P 4650 3250
-F 0 "#PWR62" H 4650 3100 50  0001 C CNN
+F 0 "#PWR066" H 4650 3100 50  0001 C CNN
 F 1 "+BATT" H 4650 3390 50  0000 C CNN
 F 2 "" H 4650 3250 50  0001 C CNN
@@
 	4650 3250 4650 3300
 $Comp
-L +BATT #PWR64
+L +BATT #PWR067
 U 1 1 5EB782BD
 P 5700 3350
-F 0 "#PWR64" H 5700 3200 50  0001 C CNN
+F 0 "#PWR067" H 5700 3200 50  0001 C CNN
 F 1 "+BATT" H 5700 3490 50  0000 C CNN
 F 2 "" H 5700 3350 50  0001 C CNN
@@
 $EndComp
 $Comp
-L +BATT #PWR49
+L +BATT #PWR068
 U 1 1 5EB78489
 P 2200 5000
-F 0 "#PWR49" H 2200 4850 50  0001 C CNN
+F 0 "#PWR068" H 2200 4850 50  0001 C CNN
 F 1 "+BATT" H 2200 5140 50  0000 C CNN
 F 2 "" H 2200 5000 50  0001 C CNN
@@
 $EndComp
 $Comp
-L +BATT #PWR56
+L +BATT #PWR069
 U 1 1 5EB78A1D
 P 3250 4800
-F 0 "#PWR56" H 3250 4650 50  0001 C CNN
+F 0 "#PWR069" H 3250 4650 50  0001 C CNN
 F 1 "+BATT" H 3250 4940 50  0000 C CNN
 F 2 "" H 3250 4800 50  0001 C CNN

Commit message: Submitted to JLCPCB 2020-07-12
Parts:
- R67: value 0R -> 47R; LCSC C17477 -> C17714
Changed lines of the file:
@@
 $Descr A4 11693 8268
 encoding utf-8
-Sheet 2 3
+Sheet 2 4
 Title ""
 Date ""
@@
 $EndComp
 $Comp
-L GND #PWR044
+L GND #PWR48
 U 1 1 5EB7DC05
 P 2200 4650
-F 0 "#PWR044" H 2200 4400 50  0001 C CNN
+F 0 "#PWR48" H 2200 4400 50  0001 C CNN
 F 1 "GND" H 2200 4500 50  0000 C CNN
 F 2 "" H 2200 4650 50  0001 C CNN
@@
 $EndComp
 $Comp
-L GND #PWR045
+L GND #PWR55
 U 1 1 5EB7DC0C
 P 3100 2550
-F 0 "#PWR045" H 3100 2300 50  0001 C CNN
+F 0 "#PWR55" H 3100 2300 50  0001 C CNN
 F 1 "GND" H 3100 2400 50  0000 C CNN
 F 2 "" H 3100 2550 50  0001 C CNN
@@
 $EndComp
 $Comp
-L GND #PWR046
+L GND #PWR44
 U 1 1 5EB7DC0E
 P 1350 3600
-F 0 "#PWR046" H 1350 3350 50  0001 C CNN
+F 0 "#PWR44" H 1350 3350 50  0001 C CNN
 F 1 "GND" H 1350 3450 50  0000 C CNN
 F 2 "" H 1350 3600 50  0001 C CNN
@@
 $EndComp
 $Comp
-L GND #PWR047
+L GND #PWR46
 U 1 1 5EB7DC14
 P 2200 2500
-F 0 "#PWR047" H 2200 2250 50  0001 C CNN
+F 0 "#PWR46" H 2200 2250 50  0001 C CNN
 F 1 "GND" H 2200 2350 50  0000 C CNN
 F 2 "" H 2200 2500 50  0001 C CNN
@@
 $EndComp
 $Comp
-L GND #PWR048
+L GND #PWR51
 U 1 1 5EB7DC1C
 P 2550 3600
-F 0 "#PWR048" H 2550 3350 50  0001 C CNN
+F 0 "#PWR51" H 2550 3350 50  0001 C CNN
 F 1 "GND" H 2550 3450 50  0000 C CNN
 F 2 "" H 2550 3600 50  0001 C CNN
@@
 $EndComp
 $Comp
-L GND #PWR049
+L GND #PWR65
 U 1 1 5EB7DC1D
 P 5700 5200
-F 0 "#PWR049" H 5700 4950 50  0001 C CNN
+F 0 "#PWR65" H 5700 4950 50  0001 C CNN
 F 1 "GND" H 5700 5050 50  0000 C CNN
 F 2 "" H 5700 5200 50  0001 C CNN
@@
 $EndComp
 $Comp
-L GND #PWR050
+L GND #PWR69
 U 1 1 5EB7DC20
 P 7200 5150
-F 0 "#PWR050" H 7200 4900 50  0001 C CNN
+F 0 "#PWR69" H 7200 4900 50  0001 C CNN
 F 1 "GND" H 7200 5000 50  0000 C CNN
 F 2 "" H 7200 5150 50  0001 C CNN
@@
 $EndComp
 $Comp
-L GND #PWR051
+L GND #PWR59
 U 1 1 5EB7DC21
 P 3500 1900
-F 0 "#PWR051" H 3500 1650 50  0001 C CNN
+F 0 "#PWR59" H 3500 1650 50  0001 C CNN
 F 1 "GND" H 3500 1750 50  0000 C CNN
 F 2 "" H 3500 1900 50  0001 C CNN
@@
 $EndComp
 $Comp
-L GND #PWR052
+L GND #PWR50
 U 1 1 5EB7DC27
 P 2200 6550
-F 0 "#PWR052" H 2200 6300 50  0001 C CNN
+F 0 "#PWR50" H 2200 6300 50  0001 C CNN
 F 1 "GND" H 2200 6400 50  0000 C CNN
 F 2 "" H 2200 6550 50  0001 C CNN
@@
 $EndComp
 $Comp
-L GND #PWR053
+L GND #PWR45
 U 1 1 5EB7DC2C
 P 1350 5500
-F 0 "#PWR053" H 1350 5250 50  0001 C CNN
+F 0 "#PWR45" H 1350 5250 50  0001 C CNN
 F 1 "GND" H 1350 5350 50  0000 C CNN
 F 2 "" H 1350 5500 50  0001 C CNN
@@
 $EndComp
 $Comp
-L GND #PWR054
+L GND #PWR52
 U 1 1 5EB7DC2F
 P 2550 5500
-F 0 "#PWR054" H 2550 5250 50  0001 C CNN
+F 0 "#PWR52" H 2550 5250 50  0001 C CNN
 F 1 "GND" H 2550 5350 50  0000 C CNN
 F 2 "" H 2550 5500 50  0001 C CNN
@@
 	3550 5600 3550 5400
 $Comp
-L GND #PWR055
+L GND #PWR57
 U 1 1 5EB7DC31
 P 3250 5850
-F 0 "#PWR055" H 3250 5600 50  0001 C CNN
+F 0 "#PWR57" H 3250 5600 50  0001 C CNN
 F 1 "GND" H 3250 5700 50  0000 C CNN
 F 2 "" H 3250 5850 50  0001 C CNN
@@
 	3650 5600 3550 5600
 $Comp
-L GND #PWR056
+L GND #PWR61
 U 1 1 5EB7DC32
 P 3950 5850
-F 0 "#PWR056" H 3950 5600 50  0001 C CNN
+F 0 "#PWR61" H 3950 5600 50  0001 C CNN
 F 1 "GND" H 3950 5700 50  0000 C CNN
 F 2 "" H 3950 5850 50  0001 C CNN
@@
 	6050 3850 6050 3750
 $Comp
-L GND #PWR057
+L GND #PWR66
 U 1 1 5EB7DC3C
 P 6050 3850
-F 0 "#PWR057" H 6050 3600 50  0001 C CNN
+F 0 "#PWR66" H 6050 3600 50  0001 C CNN
 F 1 "GND" H 6050 3700 50  0000 C CNN
 F 2 "" H 6050 3850 50  0001 C CNN
@@
 	2900 5200 2900 5100
 $Comp
-L GND #PWR058
+L GND #PWR53
 U 1 1 5EB7DC3E
 P 2900 5200
-F 0 "#PWR058" H 2900 4950 50  0001 C CNN
+F 0 "#PWR53" H 2900 4950 50  0001 C CNN
 F 1 "GND" H 2900 5050 50  0000 C CNN
 F 2 "" H 2900 5200 50  0001 C CNN
@@
 Connection ~ 4650 3650
 $Comp
-L GND #PWR059
+L GND #PWR63
 U 1 1 5EB7DC46
 P 5000 3700
-F 0 "#PWR059" H 5000 3450 50  0001 C CNN
+F 0 "#PWR63" H 5000 3450 50  0001 C CNN
 F 1 "GND" H 5000 3550 50  0000 C CNN
 F 2 "" H 5000 3700 50  0001 C CNN
@@
 Connection ~ 3350 3650
 $Comp
-L GND #PWR060
+L GND #PWR60
 U 1 1 5EB7DC4A
 P 3700 3700
-F 0 "#PWR060" H 3700 3450 50  0001 C CNN
+F 0 "#PWR60" H 3700 3450 50  0001 C CNN
 F 1 "GND" H 3700 3550 50  0000 C CNN
 F 2 "" H 3700 3700 50  0001 C CNN
@@
 $EndComp
 $Comp
-L GND #PWR061
+L GND #PWR67
 U 1 1 5EB7DC53
 P 6350 5200
-F 0 "#PWR061" H 6350 4950 50  0001 C CNN
+F 0 "#PWR67" H 6350 4950 50  0001 C CNN
 F 1 "GND" H 6350 5050 50  0000 C CNN
 F 2 "" H 6350 5200 50  0001 C CNN
@@
 $EndComp
 $Comp
-L GND #PWR062
+L GND #PWR68
 U 1 1 5EB7DC55
 P 6800 5200
-F 0 "#PWR062" H 6800 4950 50  0001 C CNN
+F 0 "#PWR68" H 6800 4950 50  0001 C CNN
 F 1 "GND" H 6800 5050 50  0000 C CNN
 F 2 "" H 6800 5200 50  0001 C CNN
@@
 P 6550 4650
 F 0 "R67" V 6630 4650 50  0000 C CNN
-F 1 "0R" V 6550 4650 50  0000 C CNN
+F 1 "47R" V 6550 4650 50  0000 C CNN
 F 2 "Resistors_SMD:R_0805_HandSoldering" V 6480 4650 50  0001 C CNN
 F 3 "" H 6550 4650 50  0001 C CNN
-F 4 "C17477" V 6550 4650 60  0001 C CNN "LCSC"
+F 4 "C17714" V 6550 4650 60  0001 C CNN "LCSC"
 	1    6550 4650
 	0    -1   -1   0
@@
 	5050 4250 5000 4250
 $Comp
-L +BATT #PWR063
+L +BATT #PWR54
 U 1 1 5EB77B79
 P 3100 1500
-F 0 "#PWR063" H 3100 1350 50  0001 C CNN
+F 0 "#PWR54" H 3100 1350 50  0001 C CNN
 F 1 "+BATT" H 3100 1640 50  0000 C CNN
 F 2 "" H 3100 1500 50  0001 C CNN
@@
 $EndComp
 $Comp
-L +BATT #PWR064
+L +BATT #PWR47
 U 1 1 5EB77C65
 P 2200 3050
-F 0 "#PWR064" H 2200 2900 50  0001 C CNN
+F 0 "#PWR47" H 2200 2900 50  0001 C CNN
 F 1 "+BATT" H 2200 3190 50  0000 C CNN
 F 2 "" H 2200 3050 50  0001 C CNN
@@
 	2200 3050 2200 3100
 $Comp
-L +BATT #PWR065
+L +BATT #PWR58
 U 1 1 5EB77FC8
 P 3350 3300
-F 0 "#PWR065" H 3350 3150 50  0001 C CNN
+F 0 "#PWR58" H 3350 3150 50  0001 C CNN
 F 1 "+BATT" H 3350 3440 50  0000 C CNN
 F 2 "" H 3350 3300 50  0001 C CNN
@@
 $EndComp
 $Comp
-L +BATT #PWR066
+L +BATT #PWR62
 U 1 1 5EB78125
 P 4650 3250
-F 0 "#PWR066" H 4650 3100 50  0001 C CNN
+F 0 "#PWR62" H 4650 3100 50  0001 C CNN
 F 1 "+BATT" H 4650 3390 50  0000 C CNN
 F 2 "" H 4650 3250 50  0001 C CNN
@@
 	4650 3250 4650 3300
 $Comp
-L +BATT #PWR067
+L +BATT #PWR64
 U 1 1 5EB782BD
 P 5700 3350
-F 0 "#PWR067" H 5700 3200 50  0001 C CNN
+F 0 "#PWR64" H 5700 3200 50  0001 C CNN
 F 1 "+BATT" H 5700 3490 50  0000 C CNN
 F 2 "" H 5700 3350 50  0001 C CNN
@@
 $EndComp
 $Comp
-L +BATT #PWR068
+L +BATT #PWR49
 U 1 1 5EB78489
 P 2200 5000
-F 0 "#PWR068" H 2200 4850 50  0001 C CNN
+F 0 "#PWR49" H 2200 4850 50  0001 C CNN
 F 1 "+BATT" H 2200 5140 50  0000 C CNN
 F 2 "" H 2200 5000 50  0001 C CNN
@@
 $EndComp
 $Comp
-L +BATT #PWR069
+L +BATT #PWR56
 U 1 1 5EB78A1D
 P 3250 4800
-F 0 "#PWR069" H 3250 4650 50  0001 C CNN
+F 0 "#PWR56" H 3250 4650 50  0001 C CNN
 F 1 "+BATT" H 3250 4940 50  0000 C CNN
 F 2 "" H 3250 4800 50  0001 C CNN
