File: RFUtilityKnife.kicad_pcb (KiCad board)
At the start: 2 copper layers, 100 x 103 mm, 334 parts, among them J1 Conn_01x01, J10 Conn_01x01, J100 Conn_01x01, J101 Conn_01x01, J102 Conn_01x01, J103 Conn_01x01, J104 Conn_01x01, J105 Conn_01x01, J106 Conn_01x01, J107 Conn_01x01, J108 Conn_01x01, J109 Conn_01x01, J11 Conn_01x01, J110 Conn_01x01, J111 Conn_01x01, J112 Conn_01x01, J113 Conn_01x01, J114 Conn_01x01, J115 Conn_01x01, J116 Conn_01x01, J117 Conn_01x01, J118 Conn_01x01, J119 Conn_01x01, J12 Conn_01x01, J120 Conn_01x01, J121 Conn_01x01, J122 Conn_01x01, J123 Conn_01x01, J124 Conn_01x01, J125 Conn_01x01, J126 Conn_Coaxial, J127 Conn_Coaxial, J128 Conn_01x01, J129 Conn_01x01, J13 Conn_01x01, J130 Conn_01x01, J131 Conn_01x01, J14 Conn_01x01, J15 Conn_01x01, J16 Conn_01x01, J17 Conn_01x01, J18 Conn_Coaxial, J19 Conn_01x01, J2 Barrel_Jack, J20 Conn_01x01, J21 Conn_01x01, J22 Conn_01x01, J23 Conn_01x01, J24 Conn_Coaxial, J25 Conn_Coaxial, J26 Conn_01x01, J27 Conn_01x01, J28 Conn_01x01, J29 Conn_01x01, J3 Conn_Coaxial, J30 Conn_01x01, J31 Conn_01x01, J32 Conn_01x01, J33 Conn_01x01, J34 Conn_01x01, J35 Conn_01x01, J36 Conn_01x01, J37 Conn_01x01, J38 Conn_01x01, J39 Conn_01x01, J4 Conn_Coaxial, J40 Conn_01x01, J41 Conn_01x01, J42 Conn_01x01, J43 Conn_01x01, J44 Conn_01x01, J45 Conn_01x01, J46 Conn_01x01, J47 Conn_01x01, J48 Conn_01x01, J49 Conn_01x01, J5 Conn_01x01, J50 Conn_01x01, J51 Conn_01x01, J52 Conn_01x01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

Commit message: JLCPCB order 2020-05-20
Parts:
- removed J113, J125: Conn_01x01, RFUtilityKnife:BigSlot
- removed L1: Ferrite_Bead, Inductors_SMD:L_0805_HandSoldering
- added RV3: 10k, Potentiometers:Potentiometer_Triwood_RM-065, F.Cu at (101.0, 93.9)
- R10, R106, R2, R24, R31, R43, R44, R62: value 220R -> 22R
- R100, R104: value 51R -> 100R
- R21: value 47k -> 10k
- R22: value 220R -> 100R
- R74, R75, R76, R86: value 220R -> 47R
- moved R21 5.83 mm to (114.3, 89.9)
- moved C10 5.32 mm to (106.5, 89.9), turned to 0 degrees
- moved Q4 5.05 mm to (106.7, 92.4), turned to 270 degrees
- moved R23 4.96 mm to (118.3, 86.1)
- moved Q5 4.45 mm to (117.2, 90.4)
- moved C14 4.29 mm to (116.3, 86.3)
- moved R22 3.89 mm to (120.1, 87.9), turned to 270 degrees
- moved JP3 3.40 mm to (82.9, 90.4), turned to 90 degrees
- moved C11 3.04 mm to (102.0, 84.0)
- moved C12 3.04 mm to (112.8, 79.4)
- moved C13 3.04 mm to (110.9, 91.3)
- moved C15 3.04 mm to (123.9, 91.3)
- moved C16 3.04 mm to (122.7, 75.0)
- moved C17 3.04 mm to (131.9, 92.6)
- moved C18 3.04 mm to (132.1, 88.0)
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Connections:
- Q5 pad 1: Net-(Q5-Pad1) -> Net-(C13-Pad1)
- Q5 pad 3: Net-(C14-Pad2) -> Net-(Q5-Pad3)
- R21 pad 1: Net-(Q5-Pad1) -> Net-(C13-Pad1)
- R22 pad 1: Net-(Q5-Pad1) -> Net-(C14-Pad2)
- R22 pad 2: Net-(C13-Pad1) -> Net-(Q5-Pad3)
Routing:
- net GND: track 421.4 -> 1051.2 mm, vias 210 -> 431
- net Net-(C16-Pad2): track 89.5 -> 101.0 mm
- net Net-(Q26-Pad2): track 6.84 -> 2.31 mm, vias 3 -> 0
- net Net-(Q5-Pad1): track 3.74 -> 0.00 mm
- net Net-(C10-Pad1): track 4.20 -> 7.61 mm
- net Net-(Q5-Pad3): track 0.00 -> 2.96 mm
- net Net-(C40-Pad2): track 38.6 -> 35.9 mm
- net Net-(C13-Pad1): track 2.19 -> 4.15 mm
- net Net-(C15-Pad2): track 3.67 -> 4.67 mm
- net Net-(C43-Pad1): track 20.4 -> 21.3 mm
- net Net-(C44-Pad1): track 6.90 -> 6.21 mm
- net Net-(C53-Pad2): track 4.37 -> 4.94 mm
- net Net-(C39-Pad2): track 6.49 -> 5.94 mm
Other:
- board size 100 x 103 mm -> 100 x 100 mm

Commit message: Real actual accepted for production by JLCPCB files, you cant fault a guy for trying
Parts:
- removed J102, J103, J104, J105, J106, J107, J108, J109, J110, J111, J112, J114, J115, J116, J117, J118, J119, J120, J121, J122, J123, J124, J19, J20, J21, J22, J23, J26, J27, J28, J29, J30, J31, J32, J33, J34, J35, J36, J37, J38, J39, J40, J41, J42, J43, J46, J47, J50, J51, J52, J54, J55, J56, J57, J58, J61, J62, J64, J66, J67, J68, J69, J73, J74, J75, J76, J77, J78, J79, J80, J81, J82, J83, J84, J85, J86, J87, J88, J89, J90, J91: Conn_01x01, RFUtilityKnife:BigSlot
- C23: value 10 nF -> 1 pF
- moved C11 12.6 mm to (101.0, 71.4), turned to 270 degrees
- moved J70 5.03 mm to (111.4, 37.1)
- moved J72 3.86 mm to (114.0, 43.0)
- moved J71 3.23 mm to (107.0, 43.0)
- moved C1 3.00 mm to (109.5, 41.0)
- moved J1 3.00 mm to (104.9, 41.0)
- moved J15 3.00 mm to (104.8, 33.9)
- moved R2 3.00 mm to (114.2, 41.0)
- moved R3 3.00 mm to (115.8, 37.7)
- moved J59 2.55 mm to (101.5, 34.5)
- moved J2 2.30 mm to (101.3, 78.6)
- moved C24 2.06 mm to (107.7, 124.2)
- moved C25 2.06 mm to (108.0, 113.5)
- moved C26 2.06 mm to (117.1, 120.4)
- moved C27 2.06 mm to (121.9, 124.2)
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Routing:
- net Net-(C11-Pad2): track 16.0 -> 12.2 mm
- net Net-(Q1-Pad1): track 4.04 -> 4.62 mm
- net Net-(C10-Pad1): track 7.61 -> 7.04 mm
- net +9V: track 34.7 -> 34.1 mm
- net GND: track 1051.2 -> 1050.8 mm, vias 431 -> 432

Commit message: Submitted to JLCPCB 2020-07-12
Parts:
- removed J92, J94, J97: Conn_Coaxial, RFUtilityKnife:Amphenol_RF_SMA_132289
- removed JP1, JP2, JP3, JP4: Jumper_NO_Small, Pin_Headers:Pin_Header_Straight_1x02_Pitch2.54mm
- removed Q20, Q21, Q22, Q8: 2SC3356, TO_SOT_Packages_SMD:SOT-23
- removed R100, R85, R87: 100R, Resistors_SMD:R_0805_HandSoldering
- removed R84: 10R, Resistors_SMD:R_0805_HandSoldering
- removed RV2: 10k, Potentiometers:Potentiometer_Triwood_RM-065
- added C50: 15 pF, Capacitors_SMD:C_0805_HandSoldering, F.Cu at (123.9, 93.3)
- added C51: 15 pF, Capacitors_SMD:C_0805_HandSoldering, F.Cu at (88.9, 53.2)
- added C52: 15 pF, Capacitors_SMD:C_0805_HandSoldering, F.Cu at (128.3, 47.4)
- added C60: 100 pF, Capacitors_SMD:C_0805_HandSoldering, F.Cu at (153.5, 81.9)
- added C61: 2.2 uF, Capacitors_SMD:C_0805_HandSoldering, F.Cu at (155.5, 70.5)
- added C62: 2.2 uF, Capacitors_SMD:C_0805_HandSoldering, F.Cu at (128.3, 71.8)
- added C63: 2.2 uF, Capacitors_SMD:C_0805_HandSoldering, F.Cu at (130.3, 71.8)
- added C64: 100 pF, Capacitors_SMD:C_0805_HandSoldering, F.Cu at (109.3, 88.9)
- added C65: 22 uF, Capacitors_SMD:C_0805_HandSoldering, F.Cu at (78.1, 89.2)
- added C66: 10 nF, Capacitors_SMD:C_0805_HandSoldering, F.Cu at (66.5, 105.8)
- added D8: D_Zener, Diodes_SMD:D_MiniMELF, F.Cu at (109.6, 92.6)
- added D9: US1MG, Diodes_SMD:D_SMA_Handsoldering, F.Cu at (140.4, 71.4)
- added J19: Conn_01x01, RFUtilityKnife:PadHole, F.Cu at (58.3, 105.1)
- added J20: Conn_01x01, RFUtilityKnife:PadHole, F.Cu at (63.1, 111.7)
- added J21: Conn_01x01, RFUtilityKnife:PadHole, F.Cu at (63.0, 105.1)
- added J22: Barrel_Jack, Connectors:BARREL_JACK, F.Cu at (65.3, 77.7)
- added J23: Barrel_Jack, Connectors:BARREL_JACK, F.Cu at (65.5, 44.7)
- added J26: Conn_01x01, RFUtilityKnife:BigSlot, F.Cu at (137.2, 34.4)
- added J27: Conn_01x01, RFUtilityKnife:BigSlot, F.Cu at (130.3, 34.4)
- added J28: Conn_01x01, RFUtilityKnife:BigSlot, F.Cu at (137.1, 50.5)
- added J29: Conn_01x01, RFUtilityKnife:BigSlot, F.Cu at (130.2, 50.5)
- added J30: Conn_01x01, RFUtilityKnife:BigSlot, F.Cu at (138.3, 130.1)
- added J31: Conn_01x01, RFUtilityKnife:BigSlot, F.Cu at (138.2, 103.8)
- added J32: Conn_01x01, RFUtilityKnife:BigSlot, F.Cu at (145.9, 130.1)
- added J33: Conn_01x01, RFUtilityKnife:BigSlot, F.Cu at (145.7, 103.8)
- added JP5: Jumper_NC_Dual, Pin_Headers:Pin_Header_Straight_1x03_Pitch2.54mm, F.Cu at (97.3, 87.1)
- added L1: 10 uH, Inductors_SMD:L_7.3x7.3_H4.5, F.Cu at (149.5, 72.7)
- added Q24: MMBT5551, TO_SOT_Packages_SMD:SOT-23, F.Cu at (148.4, 84.9)
- added Q25: MMBT5551, TO_SOT_Packages_SMD:SOT-23, F.Cu at (142.7, 75.2)
- added R92: 56R, Resistors_SMD:R_0805_HandSoldering, F.Cu at (63.7, 60.6)
- added R93: 1k, Resistors_SMD:R_0805_HandSoldering, F.Cu at (155.4, 75.4)
- added R94: 10k, Resistors_SMD:R_0805_HandSoldering, F.Cu at (151.8, 79.1)
- added R95: 1k, Resistors_SMD:R_0805_HandSoldering, F.Cu at (141.5, 79.1)
- added R96: 47k, Resistors_SMD:R_0805_HandSoldering, F.Cu at (132.4, 71.7)
- added R97: 1k, Resistors_SMD:R_0805_HandSoldering, F.Cu at (134.6, 71.7)
- added U2: NE555, Housings_SOIC:SOIC-8_3.9x4.9mm_Pitch1.27mm, F.Cu at (147.0, 80.3)
- added U3: LM78M05_TO252, TO_SOT_Packages_SMD:TO-252-3_TabPin2, F.Cu at (71.3, 88.1)
- C22: value 10 nF -> 1 pF
- C23: value 1 pF -> 10 nF; footprint Capacitors_SMD:C_0603 -> Capacitors_SMD:C_0805_HandSoldering
- C39, C44: value 10 nF -> 100 nF
- C42: value 100 nF -> 10 nF
- J4: value Conn_Coaxial -> Conn_01x01; footprint RFUtilityKnife:Amphenol_RF_SMA_132289 -> RFUtilityKnife:PadHole
- R101, R24: value 22R -> 220R
- R111, R17, R38, R67: value 0R -> 47R
- R19: value 1k -> 470R
- R20: value 2k2 -> 100R
- R21, R98: value 10k -> 47k
- R22: value 100R -> 22R
- R32: value 1k -> 56R
- R37: value 51R -> 47R; footprint Resistors_SMD:R_0603 -> Resistors_SMD:R_0805_HandSoldering
- R40: value 100R -> 220R; footprint Resistors_SMD:R_0603 -> Resistors_SMD:R_0805_HandSoldering
- R41: value 68R -> 1k5; footprint Resistors_SMD:R_0603 -> Resistors_SMD:R_0805_HandSoldering
- R42: value 100R -> 2k2; footprint Resistors_SMD:R_0603 -> Resistors_SMD:R_0805_HandSoldering
- R69, R79: value 10k -> 1k5
- R70, R83: value 10k -> 220R
- R72: value 10k -> 10R
- R74: value 47R -> 22R
- R75: value 47R -> 220R
- R76: value 47R -> 1k5
- R78: value 100R -> 2k2
- R81: value 220R -> 10k
- R82: value 22R -> 10R
- R89: value NC -> 100k
- R90: value 0R -> 22R
- RV1: value 10k -> 1k
- moved J4 101.2 mm to (58.3, 111.7)
- moved R89 86.4 mm to (155.5, 80.4)
- moved R37 86.3 mm to (59.5, 107.6), turned to 180 degrees
- moved R42 82.8 mm to (71.0, 102.1), turned to 180 degrees
- moved R40 76.3 mm to (73.0, 98.6), turned to 180 degrees
- moved R41 76.1 mm to (75.8, 102.1)
- moved R32 66.6 mm to (63.4, 95.7), turned to 90 degrees
- moved J96 45.7 mm to (80.0, 129.2), turned to 270 degrees
- moved C22 36.3 mm to (108.2, 96.1), turned to 0 degrees
- moved C23 35.1 mm to (109.3, 87.0), turned to 180 degrees
- moved C43 31.2 mm to (79.8, 124.3), turned to 90 degrees
- moved C41 26.6 mm to (76.4, 96.7), turned to 180 degrees
- moved R77 26.4 mm to (80.5, 98.5), turned to 0 degrees
- moved J95 25.9 mm to (59.7, 96.9)
- moved J93 24.8 mm to (60.0, 120.2), turned to 180 degrees
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Connections:
- C10 pad 2: GND -> Net-(C10-Pad2)
- C16 pad 2: Net-(C16-Pad2) -> NOISEPOWER
- C19 pad 2: Net-(C16-Pad2) -> NOISEPOWER
- C22 pad 2: Net-(C22-Pad2) -> Net-(C13-Pad2)
- C23 pad 2: Net-(C23-Pad2) -> Net-(C10-Pad1)
- C39 pad 1: Net-(C39-Pad1) -> GND
- C42 pad 1: GND -> Net-(C42-Pad1)
- C44 pad 1: Net-(C44-Pad1) -> GND
- D3 pad 2: Net-(C16-Pad2) -> NOISEPOWER
- D4 pad 2: Net-(C16-Pad2) -> NOISEPOWER
- J101 pad 1: GND -> Net-(C65-Pad2)
- J93 pad 1: Net-(C39-Pad2) -> Net-(J4-Pad1)
- J98 pad 1: MIXERVCC -> Net-(J100-Pad1)
- J99 pad 1: Net-(J100-Pad1) -> GND
- Q16 pad 1: Net-(Q16-Pad1) -> Net-(C66-Pad1)
- Q17 pad 2: Net-(Q17-Pad2) -> Net-(C37-Pad2)
- Q17 pad 3: Net-(Q16-Pad2) -> Net-(C41-Pad2)
- Q18 pad 1: Net-(Q18-Pad1) -> Net-(C38-Pad1)
- Q18 pad 3: Net-(Q18-Pad3) -> Net-(C42-Pad2)
- Q19 pad 1: Net-(Q18-Pad1) -> Net-(Q19-Pad1)
- Q19 pad 3: Net-(Q16-Pad3) -> Net-(C44-Pad2)
- Q23 pad 1: Net-(Q22-Pad1) -> Net-(C37-Pad1)
- Q23 pad 2: GND -> Net-(Q23-Pad2)
- Q23 pad 3: Net-(Q23-Pad3) -> Net-(Q16-Pad2)
- Q26 pad 2: Net-(Q26-Pad2) -> Net-(C55-Pad2)
- Q26 pad 3: Net-(C55-Pad2) -> Net-(C54-Pad1)
- Q4 pad 1: Net-(C13-Pad2) -> GND
- Q4 pad 2: Net-(C10-Pad1) -> Net-(C13-Pad2)
- Q5 pad 1: Net-(C13-Pad1) -> Net-(Q5-Pad1)
- Q5 pad 3: Net-(Q5-Pad3) -> Net-(C14-Pad2)
- R101 pad 2: Net-(Q26-Pad2) -> Net-(C55-Pad2)
- R19 pad 1: GND -> Net-(C13-Pad2)
- R19 pad 2: Net-(C13-Pad2) -> Net-(R19-Pad2)
- R20 pad 1: Net-(C12-Pad2) -> NOISEPOWER
- R20 pad 2: GND -> Net-(C12-Pad2)
- R21 pad 1: Net-(C13-Pad1) -> Net-(C14-Pad2)
- R21 pad 2: Net-(C14-Pad2) -> Net-(Q5-Pad1)
- R22 pad 1: Net-(C14-Pad2) -> Net-(Q5-Pad1)
- R22 pad 2: Net-(Q5-Pad3) -> Net-(C13-Pad1)
- R23 pad 2: Net-(C16-Pad2) -> NOISEPOWER
- R25 pad 1: Net-(C16-Pad2) -> Net-(C12-Pad2)
- R25 pad 2: Net-(C12-Pad2) -> GND
- R27 pad 2: Net-(C16-Pad2) -> NOISEPOWER
- R32 pad 1: Net-(C16-Pad2) -> Net-(C40-Pad2)
- R32 pad 2: Net-(R32-Pad2) -> GND
- R34 pad 2: Net-(C16-Pad2) -> NOISEPOWER
- R37 pad 1: Net-(C22-Pad2) -> GND
- R37 pad 2: Net-(C23-Pad2) -> Net-(J19-Pad1)
- R40 pad 1: Net-(Q8-Pad1) -> GND
- R40 pad 2: GND -> Net-(C37-Pad2)
- R41 pad 1: Net-(J4-Pad1) -> Net-(Q16-Pad3)
- R41 pad 2: Net-(Q8-Pad1) -> Net-(C66-Pad1)
- R42 pad 1: Net-(J4-Pad1) -> Net-(C66-Pad1)
- R42 pad 2: GND -> Net-(C37-Pad1)
- R69 pad 1: MIXERVCC -> Net-(C37-Pad1)
- R69 pad 2: Net-(C38-Pad1) -> GND
- R70 pad 1: Net-(C38-Pad1) -> Net-(Q16-Pad3)
- R70 pad 2: GND -> Net-(C39-Pad2)
- R71 pad 1: MIXERVCC -> Net-(C41-Pad2)
- R71 pad 2: Net-(C37-Pad1) -> Net-(Q17-Pad1)
- R72 pad 1: Net-(C37-Pad1) -> Net-(C39-Pad2)
- R72 pad 2: GND -> MIXERVCC
- R73 pad 1: Net-(C39-Pad1) -> Net-(C42-Pad1)
- R73 pad 2: Net-(Q16-Pad3) -> Net-(Q19-Pad1)
- R74 pad 1: Net-(Q16-Pad1) -> GND
- R74 pad 2: Net-(C37-Pad1) -> Net-(Q23-Pad2)
- R75 pad 1: Net-(Q18-Pad1) -> Net-(C42-Pad2)
- R75 pad 2: Net-(C38-Pad1) -> Net-(C39-Pad2)
- R76 pad 1: Net-(Q17-Pad1) -> Net-(C42-Pad2)
- R76 pad 2: Net-(C40-Pad1) -> Net-(C38-Pad1)
- R78 pad 1: Net-(Q16-Pad3) -> Net-(C38-Pad1)
- R78 pad 2: Net-(C41-Pad2) -> Net-(R78-Pad2)
- R79 pad 1: Net-(Q16-Pad2) -> Net-(R78-Pad2)
- R79 pad 2: Net-(Q17-Pad1) -> GND
- R80 pad 1: Net-(Q23-Pad3) -> Net-(Q17-Pad1)
- R80 pad 2: Net-(Q17-Pad2) -> Net-(C40-Pad1)
- R81 pad 1: Net-(Q22-Pad1) -> Net-(C44-Pad2)
- R81 pad 2: MIXERVCC -> Net-(Q19-Pad1)
- R82 pad 1: Net-(Q20-Pad2) -> Net-(C44-Pad2)
- R82 pad 2: Net-(Q23-Pad3) -> MIXERVCC
- R83 pad 1: Net-(Q19-Pad2) -> GND
- R83 pad 2: Net-(Q20-Pad1) -> Net-(Q19-Pad2)
- R86 pad 2: Net-(Q20-Pad1) -> Net-(Q19-Pad2)
- R89 pad 1: Net-(C53-Pad1) -> NOISEPOWER
- R89 pad 2: GND -> Net-(Q24-Pad3)
- R98 pad 1: Net-(C55-Pad2) -> Net-(C54-Pad1)
- RV1 pad 1: Net-(C12-Pad2) -> GND
- RV1 pad 2: Net-(C12-Pad2) -> GND
- RV1 pad 3: Net-(C16-Pad2) -> Net-(C12-Pad2)
- RV3 pad 1: Net-(C10-Pad1) -> Net-(R19-Pad2)
- RV3 pad 2: Net-(C16-Pad2) -> Net-(C10-Pad2)
- RV3 pad 3: Net-(C16-Pad2) -> Net-(C10-Pad2)
- U1 pad 2: Net-(C16-Pad2) -> NOISEPOWER
Routing:
- net GND: track 1050.8 -> 895.3 mm, vias 432 -> 388
- net NOISEPOWER: track 0.00 -> 140.0 mm
- net Net-(C16-Pad2): track 101.1 -> 0.00 mm
- net HIGHVOLTAGE: track 0.00 -> 68.0 mm
- net Net-(J100-Pad1): track 3.83 -> 36.9 mm
- net Net-(C40-Pad2): track 35.9 -> 6.02 mm
- net Net-(Q24-Pad1): track 0.00 -> 22.2 mm
- net Net-(C10-Pad2): track 0.00 -> 20.2 mm
- net Net-(C43-Pad1): track 21.3 -> 3.63 mm
- net MIXERVCC: track 78.1 -> 60.8 mm
- net Net-(Q18-Pad1): track 15.4 -> 0.00 mm
- net Net-(Q18-Pad3): track 14.1 -> 0.00 mm
- net Net-(Q16-Pad1): track 14.1 -> 0.00 mm
- net Net-(Q19-Pad2): track 16.0 -> 3.72 mm
- net Net-(C22-Pad2): track 11.8 -> 0.00 mm
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Other:
- board text added: "1"
- board text added: "LM317"
- board text added: "LM555"
- board text added: "LO"
- board text added: "MIX OUT"
- board text removed: "LO+"
- board text removed: "LO-"
- board text removed: "OUT+"
- board text removed: "OUT-"
- board text removed: "RF+"
- board text removed: "RF-"
- board text removed: "SERIES UNAMPLIFIED NOISE SOURCE"
- board text removed: "SHUNT AMPLIFIED NOISE SOURCE"
