File: RFUtilityKnife.sch (KiCad schematic (older format))
At the start: 187 parts, among them J1 Conn_01x01, J102 Conn_01x01, J103 Conn_01x01, J104 Conn_01x01, J105 Conn_01x01, J106 Conn_01x01, J107 Conn_01x01, J108 Conn_01x01, J109 Conn_01x01, J110 Conn_01x01, J111 Conn_01x01, J112 Conn_01x01, J113 Conn_01x01, J114 Conn_01x01, J115 Conn_01x01, J116 Conn_01x01, J117 Conn_01x01, J118 Conn_01x01, J119 Conn_01x01, J120 Conn_01x01, J121 Conn_01x01, J122 Conn_01x01, J123 Conn_01x01, J124 Conn_01x01, J125 Conn_01x01, J14 Conn_01x01, J15 Conn_01x01, J19 Conn_01x01, J2 Barrel_Jack, J20 Conn_01x01, J21 Conn_01x01, J22 Conn_01x01, J23 Conn_01x01, J24 Conn_Coaxial, J25 Conn_Coaxial, J26 Conn_01x01, J27 Conn_01x01, J28 Conn_01x01, J29 Conn_01x01, J3 Conn_Coaxial, J30 Conn_01x01, J31 Conn_01x01, J32 Conn_01x01, J33 Conn_01x01, J34 Conn_01x01, J35 Conn_01x01, J36 Conn_01x01, J37 Conn_01x01, J38 Conn_01x01, J39 Conn_01x01, J4 Conn_Coaxial, J40 Conn_01x01, J41 Conn_01x01, J42 Conn_01x01, J43 Conn_01x01, J44 Conn_01x01, J45 Conn_01x01, J46 Conn_01x01, J47 Conn_01x01, J48 Conn_01x01, J49 Conn_01x01, J5 Conn_01x01, J50 Conn_01x01, J51 Conn_01x01, J52 Conn_01x01, J53 Conn_01x01, J54 Conn_01x01, J55 Conn_01x01, J56 Conn_01x01, J57 Conn_01x01, J58 Conn_01x01, J59 Conn_01x01, J60 Conn_01x01, J61 Conn_01x01, J62 Conn_01x01, J63 Conn_01x01, J64 Conn_01x01, J65 Conn_01x01, J66 Conn_01x01, J67 Conn_01x01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

Commit message: JLCPCB order 2020-05-20
Parts:
- removed J113, J125: Conn_01x01, RFUtilityKnife:BigSlot, symbol Conn_01x01
- removed L1: Ferrite_Bead, Inductors_SMD:L_0805_HandSoldering, symbol Ferrite_Bead
- added RV3: 10k, Potentiometers:Potentiometer_Triwood_RM-065, symbol POT
- C23: value 10 nF -> 1 pF
- R10, R2, R24, R31: value 220R -> 22R; LCSC C17557 -> C17561
- R21: value 47k -> 10k; LCSC C17713 -> C17414
- R22: value 220R -> 100R; LCSC C17557 -> C17408
Connections:
- net at C16.2, C19.2, D3.2 (A)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: now also RV3.2, RV3.3
- net at C10.1, Q4.2 (E): now also RV3.1
- net at C13.1: now also Q5.1 (B), R21.1; no longer R22.2
- net at C14.2, R21.2, R23.1: now also R22.1; no longer Q5.3 (C)
- new net: Q5.3 (C), R22.2
Other:
- moved on the sheet: C14, R21, R22

Commit message: Real actual accepted for production by JLCPCB files, you cant fault a guy for trying
Parts:
- removed J102, J103, J104, J105, J106, J107, J108, J109, J110, J111, J112, J114, J115, J116, J117, J118, J119, J120, J121, J122, J123, J124, J19, J20, J21, J22, J23, J26, J27, J28, J29, J30, J31, J32, J33, J34, J35, J36, J37, J38, J39, J40, J41, J42, J43, J46, J47, J50, J51, J52, J54, J55, J56, J57, J58, J61, J62, J64, J66, J67, J68, J69, J73, J74, J75, J76, J77, J78, J79, J80, J81, J82, J83, J84, J85, J86, J87, J88, J89, J90, J91: Conn_01x01, RFUtilityKnife:BigSlot, symbol Conn_01x01
Other:
- moved on the sheet: J44, J45, J48, J49, J53, J59, J60, J63, J65, J70, J71, J72

Commit message: Submitted to JLCPCB 2020-07-12
Parts:
- removed J4: Conn_Coaxial, RFUtilityKnife:Amphenol_RF_SMA_132289, symbol Conn_Coaxial
- removed Q8: 2SC3356, TO_SOT_Packages_SMD:SOT-23, symbol MMBT3904
- removed R32: 1k, Resistors_SMD:R_0805_HandSoldering, symbol R
- removed R37: 51R, Resistors_SMD:R_0603, symbol R
- removed R40, R42: 100R, Resistors_SMD:R_0603, symbol R
- removed R41: 68R, Resistors_SMD:R_0603, symbol R
- removed RV2: 10k, Potentiometers:Potentiometer_Triwood_RM-065, symbol POT
- added C50, C52: 15 pF, Capacitors_SMD:C_0805_HandSoldering, symbol C_Small
- added C64: 100 pF, Capacitors_SMD:C_0805_HandSoldering, symbol C_Small
- added D8: D_Zener, Diodes_SMD:D_MiniMELF, symbol D_Zener
- added J26, J27, J28, J29, J30, J31, J32, J33: Conn_01x01, RFUtilityKnife:BigSlot, symbol Conn_01x01
- added JP5: Jumper_NC_Dual, Pin_Headers:Pin_Header_Straight_1x03_Pitch2.54mm, symbol Jumper_NC_Dual
- C22: value 10 nF -> 1 pF; LCSC C1710 -> C14971
- C23: value 1 pF -> 10 nF; footprint Capacitors_SMD:C_0603 -> Capacitors_SMD:C_0805_HandSoldering; LCSC C23969 -> C1710
- R17, R38: value 0R -> 47R; LCSC C17477 -> C17714
- R19: value 1k -> 470R; LCSC C17513 -> C17710
- R20: value 2k2 -> 100R; LCSC C17520 -> C17408
- R21: value 10k -> 47k; LCSC C17414 -> C17713
- R22: value 100R -> 22R; LCSC C17408 -> C17561
- R24: value 22R -> 220R; LCSC C17561 -> C17557
- RV1: value 10k -> 1k
Connections:
- net GND: now also Q4.1 (B), R25.2, RV1.1, RV1.2, C50.1, C52.1, C64.1, D8.2 (A); no longer C10.2, R19.1, R20.2
- net at Q2.2 (E), R9.2: now also C52.2
- net NOISEPOWER: now reaches C16.2, C19.2, D3.2 (A), D4.2 (A), R23.2, R27.2, R34.2, U1.2 (OUT)
- net NOISEPOWER: now also R20.1, JP5.3; no longer R25.1, RV1.3, RV3.2, RV3.3
- net at C23.2: now also C10.1
- net at Q6.2 (E), R29.2: now also C50.2
- net at R22.2: now also C13.1; no longer Q5.3 (C)
- net at R21.2, R22.1: now also Q5.1 (B); no longer C14.2, R23.1
- net at C22.2: now also C13.2, Q4.2 (E), R19.1, D8.1 (K)
- new net: C12.2, R20.2, R25.1, RV1.3, U1.1 (ADJ)
- new net: R19.2, RV3.1
- new net: C14.2, Q5.3 (C), R21.1, R23.1
- new net: C10.2, C64.2, JP5.2, RV3.2, RV3.3
- new net HIGHVOLTAGE: JP5.1
Other:
- moved on the sheet: C10, C13, Q4, Q5, R19, R20, R21, R22, R24, R25, RV1, RV3
